Commit message: latest version with some meshes and URDF adaptations, for the grasp to work but I think we didn't need all of that

File: baxter_common/baxter_description/urdf/baxter.urdf (robot description, URDF)
Before this commit: robot baxter, 49 links, 48 joints
Links:
- added link l_gripper_l_finger, mass 0.00094542; collision cylinder length=0.115 radius=0.008; visual mesh filename=package://baxter_description/meshes/electric_gripper/finger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
- added link l_gripper_r_finger, mass 0.00094542; collision cylinder length=0.115 radius=0.01; visual mesh filename=package://baxter_description/meshes/electric_gripper/finger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
- added link r_gripper_l_finger, mass 0.00094542; collision cylinder length=0.115 radius=0.008; visual mesh filename=package://baxter_description/meshes/electric_gripper/finger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
- added link r_gripper_r_finger, mass 0.00094542; collision cylinder length=0.115 radius=0.01; visual mesh filename=package://baxter_description/meshes/electric_gripper/finger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
- link collision_head_link_1: geometry collision sphere radius=0.25; visual sphere radius=0.001
- link collision_head_link_2: geometry collision sphere radius=0.25; visual sphere radius=0.001
- link head: geometry collision sphere radius=0.001; visual mesh filename=package://baxter_description/meshes/head/H0.DAE scale=1 1 1
- link left_gripper_base: mass 0.0001 -> 0.28; geometry collision cylinder length=0.1 radius=0.0275; visual mesh filename=package://baxter_description/meshes/electric_gripper/electr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 scale=1 1 1
- link left_hand_accelerometer: geometry 
- link left_hand_range: geometry visual box size=0.005 0.02 0.005
- link left_lower_elbow: geometry collision cylinder length=0.18 radius=0.08; visual mesh filename=package://baxter_description/meshes/lower_elbow/E1.DAE scale=1 1 1
- link left_lower_forearm: geometry collision cylinder length=0.16 radius=0.06; visual mesh filename=package://baxter_description/meshes/lower_forearm/W1.DAE scale=1 1 1
- link left_lower_shoulder: geometry collision cylinder length=0.25 radius=0.09; visual mesh filename=package://baxter_description/meshes/lower_shoulder/S1.DAE scale=1 1 1
- link left_upper_elbow: geometry collision cylinder length=0.107 radius=0.09; visual mesh filename=package://baxter_description/meshes/upper_elbow/E0.DAE scale=1 1 1
- link left_upper_elbow_visual: geometry collision cylinder length=0.3 radius=0.09
- link left_upper_forearm: geometry collision cylinder length=0.088 radius=0.07; visual mesh filename=package://baxter_description/meshes/upper_forearm/W0.DAE scale=1 1 1
- link left_upper_forearm_visual: geometry collision cylinder length=0.272 radius=0.07
- link left_upper_shoulder: geometry collision cylinder length=0.35 radius=0.1; visual mesh filename=package://baxter_description/meshes/upper_shoulder/S0.DAE scale=1 1 1
- link left_wrist: geometry collision cylinder length=0.165 radius=0.06; visual mesh filename=package://baxter_description/meshes/wrist/W2.DAE scale=1 1 1
- link pedestal: mass 60.86397744 -> 60.864; geometry collision box size=0.82 0.83 0.28; collision cylinder length=0.11 radius=0.19
- link right_gripper_base: mass 0.0001 -> 0.28; geometry collision cylinder length=0.1 radius=0.0275; visual mesh filename=package://baxter_description/meshes/electric_gripper/electr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 scale=1 1 1
- link right_hand_accelerometer: geometry 
- link right_hand_range: geometry visual box size=0.005 0.02 0.005
- link right_lower_elbow: geometry collision cylinder length=0.18 radius=0.08; visual mesh filename=package://baxter_description/meshes/lower_elbow/E1.DAE scale=1 1 1
- link right_lower_forearm: geometry collision cylinder length=0.16 radius=0.06; visual mesh filename=package://baxter_description/meshes/lower_forearm/W1.DAE scale=1 1 1
- link right_lower_shoulder: geometry collision cylinder length=0.25 radius=0.09; visual mesh filename=package://baxter_description/meshes/lower_shoulder/S1.DAE scale=1 1 1
- link right_upper_elbow: geometry collision cylinder length=0.107 radius=0.09; visual mesh filename=package://baxter_description/meshes/upper_elbow/E0.DAE scale=1 1 1
- link right_upper_elbow_visual: geometry collision cylinder length=0.3 radius=0.09
- link right_upper_forearm: geometry collision cylinder length=0.088 radius=0.07; visual mesh filename=package://baxter_description/meshes/upper_forearm/W0.DAE scale=1 1 1
- link right_upper_forearm_visual: geometry collision cylinder length=0.272 radius=0.07
- link right_upper_shoulder: geometry collision cylinder length=0.35 radius=0.1; visual mesh filename=package://baxter_description/meshes/upper_shoulder/S0.DAE scale=1 1 1
- link right_wrist: geometry collision cylinder length=0.165 radius=0.06; visual mesh filename=package://baxter_description/meshes/wrist/W2.DAE scale=1 1 1
- link screen: geometry collision sphere radius=0.001; visual mesh filename=package://baxter_description/meshes/head/H1.DAE scale=1 1 1
- link torso: mass 35.336455 -> 35.3365; geometry collision mesh filename=package://baxter_description/meshes/torso/base_link_simple.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; visual mesh filename=package://baxter_description/meshes/torso/base_link.DAE scale=1 1 1
Joints:
- added joint l_gripper_l_finger_joint: type prismatic, parent left_gripper, child l_gripper_l_finger, origin xyz=0.0 -0.04 0.035 rpy=1.57 0 0, axis 0 0 1, limit lower=-0.0125 upper=0.0095 effort=20.0 velocity=5.0
- added joint l_gripper_r_finger_joint: type prismatic, parent left_gripper, child l_gripper_r_finger, origin xyz=0.0 0.04 0.035 rpy=1.57 0 0, axis 0 0 1, limit lower=-0.0125 upper=0.0095 effort=20.0 velocity=5.0, mimic joint=l_gripper_l_finger_joint multiplier=-1 offset=0
- added joint r_gripper_l_finger_joint: type prismatic, parent right_gripper, child r_gripper_l_finger, origin xyz=0.0 -0.04 0.035 rpy=1.57 0 0, axis 0 0 1, limit lower=-0.0125 upper=0.0095 effort=20.0 velocity=5.0
- added joint r_gripper_r_finger_joint: type prismatic, parent right_gripper, child r_gripper_r_finger, origin xyz=0.0 0.04 0.035 rpy=1.57 0 0, axis 0 0 1, limit lower=-0.0125 upper=0.0095 effort=20.0 velocity=5.0, mimic joint=r_gripper_l_finger_joint multiplier=-1 offset=0
- joint collision_head_1: axis (none) -> 0 0 0; origin xyz=0.11 0 0.75 rpy=0 0 0 -> xyz=0.11 0 0.75 rpy=0 -0 0
- joint collision_head_2: axis (none) -> 0 0 0; origin xyz=0.11 0 0.75 rpy=0 0 0 -> xyz=0.11 0 0.75 rpy=0 -0 0
- joint display_joint: axis (none) -> 0 0 0; origin xyz=0.0 -0.016 0.0 rpy=0 0 0 -> xyz=0 -0.016 0 rpy=0 -0 0
- joint dummy: axis (none) -> 0 0 0; origin xyz=0 0 0 rpy=0 0 0 -> xyz=0 0 0 rpy=0 -0 0
- joint head_camera: axis (none) -> 0 0 0; origin xyz=0.12839 0 0.06368 rpy=1.75057 0 1.57079632679 -> xyz=0.12839 0 0.06368 rpy=1.75057 3.87602e-18 1.5708
- joint head_nod: axis (none) -> 0 0 0; origin xyz=.1227 0 0 rpy=1.75057 0 1.57079632679 -> xyz=0.1227 0 0 rpy=1.75057 3.87602e-18 1.5708
- joint head_pan: limit lower=-1.57079632679 upper=1.57079632679 effort=50000 velocity=10000 -> lower=-1.5708 upper=1.5708 effort=50000 velocity=10000; origin xyz=0.06 0 0.686 rpy=0 0 0 -> xyz=0.06 0 0.686 rpy=0 -0 0
- joint left_e0: limit lower=-3.05417993878 upper=3.05417993878 effort=50.0 velocity=1.5 -> lower=-3.05418 upper=3.05418 effort=50 velocity=1.5; origin xyz=0.102 0 0 rpy=1.57079632679 0 1.57079632679 -> xyz=0.102 0 0 rpy=1.5708 -1.14194e-16 1.5708
- joint left_e0_fixed: axis 0 0 1 -> 0 0 0; origin xyz=0.107 0 0 rpy=1.57079632679 0 1.57079632679 -> xyz=0.107 0 0 rpy=1.5708 -1.14194e-16 1.5708
- joint left_e1: limit lower=-0.05 upper=2.618 effort=50.0 velocity=1.5 -> lower=-0.05 upper=2.618 effort=50 velocity=1.5; origin xyz=0.069 0 0.26242 rpy=-1.57079632679 -1.57079632679 0 -> xyz=0.069 0 0.26242 rpy=1.57078 -1.57079 -3.14158
- joint left_endpoint: axis (none) -> 0 0 0; origin xyz=0.0 0 0.025 rpy=0 0 0 -> xyz=0 0 0.045 rpy=0 -0 0
- joint left_gripper_base: axis (none) -> 0 0 0; origin xyz=0 0 0 rpy=0 0 0 -> xyz=0 0 0 rpy=0 -0 0
- joint left_hand: axis 0 0 1 -> 0 0 0; origin xyz=0 0 0.11355 rpy=0 0 0 -> xyz=0 0 0.11355 rpy=0 -0 0
- joint left_hand_accelerometer: axis (none) -> 0 0 0; origin xyz=0.00198 0.000133 -0.0146 rpy=0 0 0 -> xyz=0.00198 0.000133 -0.0146 rpy=0 -0 0
- joint left_hand_camera: axis (none) -> 0 0 0; origin xyz=0.03825 0.012 0.015355 rpy=0 0 -1.57079633 -> xyz=0.03825 0.012 0.015355 rpy=0 0 -1.5708
- joint left_hand_camera_axis: axis (none) -> 0 0 0; origin xyz=0.03825 0.012 0.015355 rpy=0 0 0 -> xyz=0.03825 0.012 0 rpy=0 -0 0
- joint left_hand_range: axis (none) -> 0 0 0; origin xyz=0.032 -0.020245 0.0288 rpy=0 -1.57079632679 -1.57079632679 -> xyz=0.032 -0.020245 0.0288 rpy=-3.14158 -1.57079 1.57078
- joint left_s0: limit lower=-1.70167993878 upper=1.70167993878 effort=50.0 velocity=1.5 -> lower=-1.70168 upper=1.70168 effort=50 velocity=1.5; origin xyz=0.055695 0 0.011038 rpy=0 0 0 -> xyz=0.055695 0 0.011038 rpy=0 -0 0
- joint left_s1: limit lower=-2.147 upper=1.047 effort=100.0 velocity=1.5 -> lower=-2.147 upper=1.047 effort=50 velocity=1.5; origin xyz=0.069 0 0.27035 rpy=-1.57079632679 0 0 -> xyz=0.069 0 0.27035 rpy=-1.5708 0 0
- joint left_torso_arm_mount: axis (none) -> 0 0 0; origin xyz=0.024645 0.219645 0.118588 rpy=0 0 0.7854 -> xyz=0.0252503 0.219489 0.109759 rpy=-0.00479639 0.00185872 0.779972
- joint left_torso_itb_fixed: axis (none) -> 0 0 0; origin xyz=-0.08897 0.15593 0.389125 rpy=-1.57079632679 3.1415 0 -> xyz=-0.08897 0.15593 0.389125 rpy=1.5708 9.26536e-05 -3.14159
- joint left_w0: limit lower=-3.059 upper=3.059 effort=15.0 velocity=4.0 -> lower=-3.059 upper=3.059 effort=15 velocity=4; origin xyz=0.10359 0 0 rpy=1.57079632679 0 1.57079632679 -> xyz=0.10359 0 0 rpy=1.5708 -1.14194e-16 1.5708
- joint left_w0_fixed: axis 0 0 1 -> 0 0 0; origin xyz=0.088 0 0 rpy=1.57079632679 0 1.57079632679 -> xyz=0.088 0 0 rpy=1.5708 -1.14194e-16 1.5708
- joint left_w0_to_itb_fixed: axis 0 0 1 -> 0 0 0; origin xyz=-0.0565 0 0.12 rpy=-1.57079632679 0 1.57079632679 -> xyz=-0.0565 0 0.12 rpy=-1.5708 1.14194e-16 1.5708
- joint left_w1: limit lower=-1.57079632679 upper=2.094 effort=15.0 velocity=4.0 -> lower=-1.5708 upper=2.094 effort=15 velocity=4; origin xyz=0.01 0 0.2707 rpy=-1.57079632679 -1.57079632679 0 -> xyz=0.01 0 0.2707 rpy=1.57078 -1.57079 -3.14158
- joint left_w2: limit lower=-3.059 upper=3.059 effort=15.0 velocity=4.0 -> lower=-3.059 upper=3.059 effort=15 velocity=4; origin xyz=0.115975 0 0 rpy=1.57079632679 0 1.57079632679 -> xyz=0.115975 0 0 rpy=1.5708 -1.14194e-16 1.5708
- joint pedestal_fixed: axis (none) -> 0 0 0; origin xyz=0.0 0.0 0.0 rpy=0 0 0 -> xyz=0 0 0 rpy=0 -0 0
- joint right_e0: limit lower=-3.05417993878 upper=3.05417993878 effort=50.0 velocity=1.5 -> lower=-3.05418 upper=3.05418 effort=50 velocity=1.5; origin xyz=0.102 0 0 rpy=1.57079632679 0 1.57079632679 -> xyz=0.102 0 0 rpy=1.5708 -1.14194e-16 1.5708
- joint right_e0_fixed: axis 0 0 1 -> 0 0 0; origin xyz=0.107 0 0 rpy=1.57079632679 0 1.57079632679 -> xyz=0.107 0 0 rpy=1.5708 -1.14194e-16 1.5708
- joint right_e1: limit lower=-0.05 upper=2.618 effort=50.0 velocity=1.5 -> lower=-0.05 upper=2.618 effort=50 velocity=1.5; origin xyz=0.069 0 0.26242 rpy=-1.57079632679 -1.57079632679 0 -> xyz=0.069 0 0.26242 rpy=1.57078 -1.57079 -3.14158
- joint right_endpoint: axis (none) -> 0 0 0; origin xyz=0.0 0 0.025 rpy=0 0 0 -> xyz=0 0 0.045 rpy=0 -0 0
- joint right_gripper_base: axis (none) -> 0 0 0; origin xyz=0 0 0 rpy=0 0 0 -> xyz=0 0 0 rpy=0 -0 0
- joint right_hand: axis 0 0 1 -> 0 0 0; origin xyz=0 0 0.11355 rpy=0 0 0 -> xyz=0 0 0.11355 rpy=0 -0 0
- joint right_hand_accelerometer: axis (none) -> 0 0 0; origin xyz=0.00198 0.000133 -0.0146 rpy=0 0 0 -> xyz=0.00198 0.000133 -0.0146 rpy=0 -0 0
- joint right_hand_camera: axis (none) -> 0 0 0; origin xyz=0.03825 0.012 0.015355 rpy=0 0 -1.57079633 -> xyz=0.03825 0.012 0.015355 rpy=0 0 -1.5708
- joint right_hand_camera_axis: axis (none) -> 0 0 0; origin xyz=0.03825 0.012 0.015355 rpy=0 0 0 -> xyz=0.03825 0.012 0 rpy=0 -0 0
- joint right_hand_range: axis (none) -> 0 0 0; origin xyz=0.032 -0.020245 0.0288 rpy=0 -1.57079632679 -1.57079632679 -> xyz=0.032 -0.020245 0.0288 rpy=-3.14158 -1.57079 1.57078
- joint right_s0: limit lower=-1.70167993878 upper=1.70167993878 effort=50.0 velocity=1.5 -> lower=-1.70168 upper=1.70168 effort=50 velocity=1.5; origin xyz=0.055695 0 0.011038 rpy=0 0 0 -> xyz=0.055695 0 0.011038 rpy=0 -0 0
- joint right_s1: limit lower=-2.147 upper=1.047 effort=100.0 velocity=1.5 -> lower=-2.147 upper=1.047 effort=50 velocity=1.5; origin xyz=0.069 0 0.27035 rpy=-1.57079632679 0 0 -> xyz=0.069 0 0.27035 rpy=-1.5708 0 0
- joint right_torso_arm_mount: axis (none) -> 0 0 0; origin xyz=0.024645 -0.219645 0.118588 rpy=0 0 -0.7854 -> xyz=0.023277 -0.21986 0.10804 rpy=0.0174986 0.00342261 -0.785584
- joint right_torso_itb_fixed: axis (none) -> 0 0 0; origin xyz=-0.08897 -0.15593 0.389125 rpy=1.57079632679 0 0 -> xyz=-0.08897 -0.15593 0.389125 rpy=1.5708 -0 0
- joint right_w0: limit lower=-3.059 upper=3.059 effort=15.0 velocity=4.0 -> lower=-3.059 upper=3.059 effort=15 velocity=4; origin xyz=0.10359 0 0 rpy=1.57079632679 0 1.57079632679 -> xyz=0.10359 0 0 rpy=1.5708 -1.14194e-16 1.5708
- joint right_w0_fixed: axis 0 0 1 -> 0 0 0; origin xyz=0.088 0 0 rpy=1.57079632679 0 1.57079632679 -> xyz=0.088 0 0 rpy=1.5708 -1.14194e-16 1.5708
- joint right_w0_to_itb_fixed: axis 0 0 1 -> 0 0 0; origin xyz=-0.0565 0 0.12 rpy=-1.57079632679 0 1.57079632679 -> xyz=-0.0565 0 0.12 rpy=-1.5708 1.14194e-16 1.5708
- joint right_w1: limit lower=-1.57079632679 upper=2.094 effort=15.0 velocity=4.0 -> lower=-1.5708 upper=2.094 effort=15 velocity=4; origin xyz=0.01 0 0.2707 rpy=-1.57079632679 -1.57079632679 0 -> xyz=0.01 0 0.2707 rpy=1.57078 -1.57079 -3.14158
- joint right_w2: limit lower=-3.059 upper=3.059 effort=15.0 velocity=4.0 -> lower=-3.059 upper=3.059 effort=15 velocity=4; origin xyz=0.115975 0 0 rpy=1.57079632679 0 1.57079632679 -> xyz=0.115975 0 0 rpy=1.5708 -1.14194e-16 1.5708
- joint sonar_s0: axis 0 0 1 -> 0 0 0; origin xyz=0.0947 0 .817 rpy=0 0 0 -> xyz=0.0947 0 0.817 rpy=0 -0 0
- joint torso_t0: axis (none) -> 0 0 0; origin xyz=0 0 0 rpy=0 0 0 -> xyz=0 0 0 rpy=0 -0 0
